File: SpiCurrent-New.sch (EAGLE design)
At the start: 58 parts, among them IC1 AD822N, IC2 AD822N, IC3 ACS758LCB-050B-PFF-T, IC4 ACS758LCB-050B-PFF-T, U1 HIP4081AIPZ

Commit message: begun layout
Parts:
- added C9: 0.1uf, rcl:C-EU050-055X075
Connections:
- net +5V: now also C9.1
- net GND: now also C9.2
Changed lines of the file:
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@@
 <part name="H7" library="holes" deviceset="MOUNT-HOLE" device="2.8"/>
 <part name="H8" library="holes" deviceset="MOUNT-HOLE" device="2.8"/>
+<part name="C9" library="rcl" deviceset="C-EU" device="050-055X075" value="0.1uf"/>
 </parts>
 <sheets>
@@
 <instance part="H7" gate="G$1" x="-45.72" y="129.54"/>
 <instance part="H8" gate="G$1" x="-45.72" y="121.92"/>
+<instance part="C9" gate="G$1" x="-88.9" y="63.5"/>
 </instances>
 <busses>
@@
 <pinref part="SUPPLY17" gate="GND" pin="GND"/>
 <wire x1="-88.9" y1="48.26" x2="-93.98" y2="48.26" width="0.1524" layer="91"/>
+<pinref part="C9" gate="G$1" pin="2"/>
+<wire x1="-88.9" y1="58.42" x2="-88.9" y2="48.26" width="0.1524" layer="91"/>
+<junction x="-88.9" y="48.26"/>
 </segment>
 <segment>
@@
 <pinref part="U$1" gate="G$1" pin="VCC"/>
 <wire x1="-93.98" y1="78.74" x2="-88.9" y2="78.74" width="0.1524" layer="91"/>
-</segment>
-<segment>
+<pinref part="C9" gate="G$1" pin="1"/>
+<wire x1="-88.9" y1="66.04" x2="-88.9" y2="78.74" width="0.1524" layer="91"/>
+<junction x="-88.9" y="78.74"/>
+</segment>
+<segment>
